File: si5351.kicad_pcb (KiCad board)
At the start: 2 copper layers, 91 x 74 mm, 60 parts, among them J1 Conn_01x07, U1 Si5351A-B-GT, Y1 Crystal_GND24

Commit message: added caps
Parts:
- removed the J1 at (236.0, 142.0)
- removed the J1 at (236.0, 92.0)
- removed the J1 at (213.0, 92.0)
- removed the J1 at (259.0, 142.0)
- removed the J1 at (213.0, 142.0)
- removed the J1 at (190.0, 142.0)
- removed the J1 at (236.0, 117.0)
- removed the J1 at (259.0, 117.0)
- removed the J1 at (213.0, 117.0)
- removed the J1 at (190.0, 117.0)
- removed the J1 at (259.0, 92.0)
- removed the R1 at (230.2, 144.5)
- removed the R1 at (230.2, 94.5)
- removed the R1 at (207.2, 94.5)
- removed the R1 at (207.2, 144.5)
- removed the R1 at (184.2, 144.5)
- removed the R1 at (253.2, 144.5)
- removed the R1 at (230.2, 119.5)
- removed the R1 at (207.2, 119.5)
- removed the R1 at (184.2, 119.5)
- removed the R1 at (253.2, 119.5)
- removed the R1 at (253.2, 94.5)
- removed the R2 at (207.2, 147.1)
- removed the R2 at (230.2, 97.1)
- removed the R2 at (207.2, 97.1)
- removed the R2 at (230.2, 147.1)
- removed the R2 at (253.2, 147.1)
- removed the R2 at (184.2, 147.1)
- removed the R2 at (207.2, 122.1)
- removed the R2 at (230.2, 122.1)
- removed the R2 at (253.2, 122.1)
- removed the R2 at (184.2, 122.1)
- removed the R2 at (253.2, 97.1)
- removed the U1 at (206.7, 155.5)
- removed the U1 at (229.7, 105.5)
- removed the U1 at (206.7, 105.5)
- removed the U1 at (183.7, 155.5)
- removed the U1 at (229.7, 155.5)
- removed the U1 at (252.7, 155.5)
- removed the U1 at (206.7, 130.5)
- removed the U1 at (183.7, 130.5)
- removed the U1 at (229.7, 130.5)
- removed the U1 at (252.7, 130.5)
- removed the U1 at (252.7, 105.5)
- removed the Y1 at (177.0, 155.5)
- removed the Y1 at (246.0, 105.5)
- removed the Y1 at (200.0, 105.5)
- removed the Y1 at (200.0, 155.5)
- removed the Y1 at (223.0, 155.5)
- removed the Y1 at (246.0, 155.5)
- removed the Y1 at (177.0, 130.5)
- removed the Y1 at (200.0, 130.5)
- removed the Y1 at (223.0, 130.5)
- removed the Y1 at (246.0, 130.5)
- removed the Y1 at (223.0, 105.5)
- added C1: 1uF, Xenir:Capacitor 1206, F.Cu at (178.8, 92.2)
- added C2: .1uF, Xenir:Capacitor 1206, F.Cu at (182.1, 92.2)
Routing:
- net (no net): track 1330.1 -> 0.00 mm
- net +3V3: track 23.8 -> 27.1 mm
- removed copper zone on F.Cu, net (none)
Other:
- board size 91 x 74 mm -> 22 x 24 mm
