File: si5351.sch (KiCad schematic (older format))
At the start: 5 parts, among them J1 Conn_01x07, U1 Si5351A-B-GT, Y1 Crystal_GND24

Commit message: gg
Parts:
- R1, R2: symbol xenir:Resistor -> si5351-rescue:Resistor-xenir
Changed lines of the file:
@@
 $EndComp
 $Comp
-L xenir:Resistor R1
+L si5351-rescue:Resistor-xenir R1
 U 1 1 63699097
 P 2100 3150
@@
 $EndComp
 $Comp
-L xenir:Resistor R2
+L si5351-rescue:Resistor-xenir R2
 U 1 1 6369A400
 P 2350 3150

Commit message: gg
Parts:
- R1, R2: symbol si5351-rescue:Resistor-xenir -> si5351-rescue:Resistor-xenir-si5351-rescue
Changed lines of the file:
@@
 $EndComp
 $Comp
-L si5351-rescue:Resistor-xenir R1
+L si5351-rescue:Resistor-xenir-si5351-rescue R1
 U 1 1 63699097
 P 2100 3150
@@
 $EndComp
 $Comp
-L si5351-rescue:Resistor-xenir R2
+L si5351-rescue:Resistor-xenir-si5351-rescue R2
 U 1 1 6369A400
 P 2350 3150

Commit message: added caps
Parts:
- added C1: 1uF, Xenir:Capacitor 1206, symbol Xenir:Capacitor
- added C2: .1uF, Xenir:Capacitor 1206, symbol Xenir:Capacitor
Connections:
- net +3V3: now also C1.1, C2.1
- net GND: now also C1.2, C2.2
Changed lines of the file:
@@
 L power:+3V3 #PWR0102
 U 1 1 636A63BD
-P 4050 2550
-F 0 "#PWR0102" H 4050 2400 50  0001 C CNN
-F 1 "+3V3" H 4065 2723 50  0000 C CNN
-F 2 "" H 4050 2550 50  0001 C CNN
-F 3 "" H 4050 2550 50  0001 C CNN
-	1    4050 2550
+P 4050 2050
+F 0 "#PWR0102" H 4050 1900 50  0001 C CNN
+F 1 "+3V3" H 4065 2223 50  0000 C CNN
+F 2 "" H 4050 2050 50  0001 C CNN
+F 3 "" H 4050 2050 50  0001 C CNN
+	1    4050 2050
 	1    0    0    -1
 $EndComp
@@
 Wire Wire Line
 	4250 2650 4050 2650
-Wire Wire Line
-	4050 2550 4050 2650
-Connection ~ 4050 2650
 Wire Wire Line
 	4050 2650 4050 2750
@@
 Text GLabel 5900 3300 2    50   Input ~ 0
 CLK0
+$Comp
+L Xenir:Capacitor C1
+U 1 1 636C1CBC
+P 3600 2350
+F 0 "C1" H 3500 2300 28  0000 C CNN
+F 1 "1uF" H 3600 2225 28  0000 C CNN
+F 2 "Xenir:Capacitor 1206" H 3600 2200 50  0001 C CNN
+F 3 "" H 3600 2200 50  0001 C CNN
+	1    3600 2350
+	0    1    1    0
+$EndComp
+$Comp
+L Xenir:Capacitor C2
+U 1 1 636C27F7
+P 3850 2350
+F 0 "C2" H 3750 2300 28  0000 C CNN
+F 1 ".1uF" H 3850 2225 28  0000 C CNN
+F 2 "Xenir:Capacitor 1206" H 3850 2200 50  0001 C CNN
+F 3 "" H 3850 2200 50  0001 C CNN
+	1    3850 2350
+	0    1    1    0
+$EndComp
+Wire Wire Line
+	3600 2200 3850 2200
+Wire Wire Line
+	3850 2200 4050 2200
+Connection ~ 3850 2200
+Wire Wire Line
+	4050 2050 4050 2200
+Wire Wire Line
+	4050 2650 4050 2200
+Connection ~ 4050 2650
+Connection ~ 4050 2200
+$Comp
+L power:GND #PWR0108
+U 1 1 636C3CCE
+P 3600 2500
+F 0 "#PWR0108" H 3600 2250 50  0001 C CNN
+F 1 "GND" H 3605 2327 50  0000 C CNN
+F 2 "" H 3600 2500 50  0001 C CNN
+F 3 "" H 3600 2500 50  0001 C CNN
+	1    3600 2500
+	1    0    0    -1
+$EndComp
+$Comp
+L power:GND #PWR0109
+U 1 1 636C405D
+P 3850 2500
+F 0 "#PWR0109" H 3850 2250 50  0001 C CNN
+F 1 "GND" H 3855 2327 50  0000 C CNN
+F 2 "" H 3850 2500 50  0001 C CNN
+F 3 "" H 3850 2500 50  0001 C CNN
+	1    3850 2500
+	1    0    0    -1
+$EndComp
 $EndSCHEMATC
